Commit message: Add config for nav2 with hunter in gazebo

File: Workspace/ros2_ws/src/hunter_ros2/hunter_gazebo/urdf/hunter_v1_ntunav_gazebo.xacro (robot description, xacro)
@@ -21,15 +21,15 @@
         </visual>
         <collision>
-            <origin xyz="0.29 0 0.05" rpy="0 0 0" />
-            <geometry>
-                <box size="0.25 0.38 0.26"/>
+            <origin xyz="0.30 0 0.05" rpy="0 0 0" />
+            <geometry>
+                <box size="0.8 0.38 0.26"/>
             </geometry>
         </collision>
-        <collision>
+        <!--collision>
             <origin xyz="-0.1 0 0.07" rpy="0 0 0" />
             <geometry>
                 <box size="0.56 0.38 0.22"/>
             </geometry>
-        </collision>
+        </collision-->
     </link>
     <!-- sensors  -->
@@ -48,4 +48,44 @@
         <origin xyz="0.43 0.0 0.62" rpy="0 0 0" />
     </joint>
+    <gazebo reference="rslidar">
+        <sensor name="lidar" type="ray">
+            <always_on>true</always_on>
+            <visualize>true</visualize>
+            <update_rate>5</update_rate>
+            <ray>
+            <scan>
+                <horizontal>
+                    <samples>360</samples>
+                    <resolution>1.000000</resolution>
+                    <min_angle>0.000000</min_angle>
+                    <max_angle>6.280000</max_angle>
+                </horizontal>
+                <!--vertical>
+                    <samples>32</samples>
+                    <resolution>1.000000</resolution>
+                    <min_angle>-0.53529248</min_angle>
+                    <max_angle>0.18622663</max_angle>
+                </vertical-->
+            </scan>
+            <range>
+                <min>0.120000</min>
+                <max>3.5</max>
+                <resolution>0.015000</resolution>
+            </range>
+            <noise>
+                <type>gaussian</type>
+                <mean>0.0</mean>
+                <stddev>0.01</stddev>
+            </noise>
+            </ray>
+            <plugin name="scan" filename="libgazebo_ros_ray_sensor.so">
+            <ros>
+                <remapping>~/out:=scan</remapping>
+            </ros>
+            <output_type>sensor_msgs/LaserScan</output_type>
+            <frame_name>rslidar</frame_name>
+            </plugin>
+        </sensor>
+    </gazebo>
     <link name="imu_link">
         <visual>
@@ -144,4 +184,46 @@
         <origin xyz="0.62 0.0 0.25" rpy="0 0 0" />
     </joint>
+    <link name="d435_front_depth_frame"/>
+    <joint name="d435_front_depth_joint" type="fixed">
+        <origin xyz="0 0 0" rpy="${-pi/2} 0 ${-pi/2}"/>
+        <parent link="d435_front_link"/>
+        <child link="d435_front_depth_frame"/>
+    </joint>
+    <gazebo reference="d435_front_link">
+    <sensor name="depth_camera" type="depth">
+        <visualize>true</visualize>
+        <update_rate>30.0</update_rate>
+        <camera name="camera">
+        <horizontal_fov>1.047198</horizontal_fov>
+        <image>
+            <width>640</width>
+            <height>480</height>
+            <format>R8G8B8</format>
+        </image>
+        <clip>
+            <near>0.05</near>
+            <far>3</far>
+        </clip>
+        </camera>
+        <plugin name="depth_camera_controller" filename="libgazebo_ros_camera.so">
+        <baseline>0.2</baseline>
+        <alwaysOn>true</alwaysOn>
+        <updateRate>0.0</updateRate>
+        <frame_name>d435_front_depth_frame</frame_name>
+        <pointCloudCutoff>0.1</pointCloudCutoff>
+        <pointCloudCutoffMax>5.0</pointCloudCutoffMax>
+        <distortionK1>0</distortionK1>
+        <distortionK2>0</distortionK2>
+        <distortionK3>0</distortionK3>
+        <distortionT1>0</distortionT1>
+        <distortionT2>0</distortionT2>
+        <CxPrime>0</CxPrime>
+        <Cx>0</Cx>
+        <Cy>0</Cy>
+        <focalLength>0</focalLength>
+        <hackBaseline>0</hackBaseline>
+        </plugin>
+    </sensor>
+    </gazebo>
     <link name="d435_rear_link">
         <visual>
@@ -394,5 +476,5 @@
         <publish_odom_tf>true</publish_odom_tf>
         <publish_wheel_tf>true</publish_wheel_tf>
-        <publish_distance>true</publish_distance>
+        <publish_distance>false</publish_distance>
         <odometry_frame>odom</odometry_frame>
         <robot_base_frame>base_link</robot_base_frame>

Commit message: Add Cafe gazebo senario

File: Workspace/ros2_ws/src/hunter_ros2/hunter_gazebo/urdf/hunter_v1_ntunav_gazebo.xacro (robot description, xacro)
@@ -12,4 +12,6 @@
     <xacro:property name="wheel_length" value="1.1653e-01" />
     <xacro:property name="wheel_radius" value="1.6459e-01" />
+	<xacro:property name="damping_value" value="10" />
+	<xacro:property name="friction_value" value="0.1" />
     <!-- Base link -->
     <link name="base_link">
@@ -26,10 +28,4 @@
             </geometry>
         </collision>
-        <!--collision>
-            <origin xyz="-0.1 0 0.07" rpy="0 0 0" />
-            <geometry>
-                <box size="0.56 0.38 0.22"/>
-            </geometry>
-        </collision-->
     </link>
     <!-- sensors  -->
@@ -249,7 +245,4 @@
         <inertial>
             <mass value="40" />
-            <!-- <mass value="50" /> -->
-            <!-- <origin xyz="-0.00065 -0.085 0.062" />
-            <inertia ixx="0.6022" ixy="-0.02364" ixz="-0.1197" iyy="1.7386" iyz="-0.001544" izz="2.0296" /> -->
             <origin xyz="0.0 0.0 0.0" />
             <inertia ixx="2.288641" ixy="0" ixz="0" iyy="5.103976" iyz="0" izz="3.431465" />
@@ -300,10 +293,4 @@
             </geometry>
         </visual>
-        <!-- <visual>
-            <origin xyz="0 0 0" rpy="0 0 0" />
-            <geometry>
-                <mesh filename="package://hunter_description/meshes/hub_shape.stl" />
-            </geometry>
-        </visual> -->
         <collision>
             <origin xyz="0 0 0" rpy="${M_PI/2} 0 0" />
@@ -352,10 +339,4 @@
             </geometry>
         </visual>
-        <!-- <visual>
-            <origin xyz="0 0 0" rpy="0 0 3.14" />
-            <geometry>
-                <mesh filename="package://hunter_description/meshes/hub_shape.stl" />
-            </geometry>
-        </visual> -->
         <collision>
             <origin xyz="0 0 0" rpy="${M_PI/2} 0 0" />
@@ -365,5 +346,5 @@
         </collision>
     </link>
-    <!--Virtual steering wheel-->
+    <!--Virtual steering wheel>
     <link name="steering_wheel_link">
         <inertial>
@@ -379,5 +360,5 @@
         <axis xyz="0 0 1" rpy="0 0 0" />
         <limit lower="-0.785" upper="0.785" effort="20" velocity="0.8" />
-    </joint>
+    </joint-->
     <!-- rear left wheel -->
     <link name="rear_left_wheel_link">
@@ -393,10 +374,4 @@
             </geometry>
         </visual>
-        <!-- <visual>
-            <origin xyz="0 0 0" rpy="0 0 3.14" />
-            <geometry>
-                <mesh filename="package://hunter_description/meshes/hub_shape.stl" />
-            </geometry>
-        </visual> -->
         <collision>
             <origin xyz="0 0 0" rpy="${M_PI/2} 0 0" />
@@ -425,10 +400,4 @@
             </geometry>
         </visual>
-        <!-- <visual>
-            <origin xyz="0 0 0" rpy="0 0 0" />
-            <geometry>
-                <mesh filename="package://hunter_description/meshes/hub_shape.stl" />
-            </geometry>
-        </visual> -->
         <collision>
             <origin xyz="0 0 0" rpy="${M_PI/2} 0 0" />
@@ -457,5 +426,5 @@
         <left_steering_joint>front_left_steering</left_steering_joint>
         <right_steering_joint>front_right_steering</right_steering_joint>
-        <steering_wheel_joint>steering_wheel</steering_wheel_joint>
+        <!--steering_wheel_joint>steering_wheel</steering_wheel_joint-->
         <!-- Max absolute steer angle for tyre in radians-->
         <!-- Any cmd_vel angular z greater than this would be capped -->
@@ -466,9 +435,9 @@
         <max_speed>1</max_speed>
         <!-- PID tuning -->
-        <left_steering_pid_gain>30 0 1</left_steering_pid_gain>
+        <left_steering_pid_gain>10 0 1</left_steering_pid_gain>
         <left_steering_i_range>0 0</left_steering_i_range>
-        <right_steering_pid_gain>30 0 1</right_steering_pid_gain>
+        <right_steering_pid_gain>10 0 1</right_steering_pid_gain>
         <right_steering_i_range>0 0</right_steering_i_range>
-        <linear_velocity_pid_gain>50 0 1</linear_velocity_pid_gain>
+        <linear_velocity_pid_gain>20 0 1</linear_velocity_pid_gain>
         <linear_velocity_i_range>0 0</linear_velocity_i_range>
         <!-- output -->

Commit message: PID modification

File: Workspace/ros2_ws/src/hunter_ros2/hunter_gazebo/urdf/hunter_v1_ntunav_gazebo.xacro (robot description, xacro)
@@ -260,5 +260,6 @@
         <child link="front_right_steer_link"/>
         <axis xyz="0 0 1" rpy="0 0 0" />
-        <limit lower="-0.785" upper="0.785" effort="20" velocity="0.8" />
+        <dynamics damping="0.0" friction="2"/>
+        <limit lower="-0.52" upper="0.52" effort="20" velocity="0.8" />
     </joint>
     <link name="front_right_steer_link">
@@ -280,4 +281,5 @@
         <child link="front_right_wheel_link"/>
         <axis xyz="0 1 0" rpy="0 0 0" />
+        <dynamics damping="0.0" friction="1.0"/>
     </joint>
     <link name="front_right_wheel_link">
@@ -306,5 +308,6 @@
         <child link="front_left_steer_link"/>
         <axis xyz="0 0 1" rpy="0 0 0" />
-        <limit lower="-0.785" upper="0.785" effort="20" velocity="0.8" />
+        <dynamics damping="0.0" friction="2"/>
+        <limit lower="-0.52" upper="0.52" effort="20" velocity="0.8" />
     </joint>
     <link name="front_left_steer_link">
@@ -326,4 +329,5 @@
         <child link="front_left_wheel_link"/>
         <axis xyz="0 1 0" rpy="0 0 0" />
+        <dynamics damping="0.0" friction="1.0"/>
     </joint>
     <link name="front_left_wheel_link">
@@ -385,4 +389,5 @@
         <parent link="base_link"/>
         <child link="rear_left_wheel_link"/>
+        <dynamics damping="0.0" friction="15"/>
         <axis xyz="0 1 0" rpy="0 0 0" />
     </joint>
@@ -411,12 +416,13 @@
         <parent link="base_link"/>
         <child link="rear_right_wheel_link"/>
+        <dynamics damping="0.0" friction="15"/>
         <axis xyz="0 1 0" rpy="0 0 0" />
     </joint>
     <gazebo>
     <plugin name='ackermann_drive' filename='libgazebo_ros_ackermann_drive.so'>
-        <ros>
+        <!--ros>
           <namespace>demo</namespace>
-        </ros>
-        <update_rate>50.0</update_rate>
+        </ros-->
+        <update_rate>100.0</update_rate>
         <!-- wheels -->
         <front_left_joint>front_left_wheel</front_left_joint>
@@ -431,18 +437,18 @@
         <max_steer>1.0</max_steer>
         <!-- Max absolute steering angle of steering wheel -->
-        <max_steering_angle>7.85</max_steering_angle>
+        <max_steering_angle>0.52</max_steering_angle>
         <!-- Max absolute linear speed in m/s -->
-        <max_speed>1</max_speed>
+        <max_speed>1.5</max_speed>
         <!-- PID tuning -->
-        <left_steering_pid_gain>10 0 1</left_steering_pid_gain>
+        <left_steering_pid_gain>1500 0 1</left_steering_pid_gain>
         <left_steering_i_range>0 0</left_steering_i_range>
-        <right_steering_pid_gain>10 0 1</right_steering_pid_gain>
+        <right_steering_pid_gain>1500 0 1</right_steering_pid_gain>
         <right_steering_i_range>0 0</right_steering_i_range>
-        <linear_velocity_pid_gain>20 0 1</linear_velocity_pid_gain>
+        <linear_velocity_pid_gain>50 0 1</linear_velocity_pid_gain>
         <linear_velocity_i_range>0 0</linear_velocity_i_range>
         <!-- output -->
         <publish_odom>true</publish_odom>
         <publish_odom_tf>true</publish_odom_tf>
-        <publish_wheel_tf>true</publish_wheel_tf>
+        <publish_wheel_tf>false</publish_wheel_tf>
         <publish_distance>false</publish_distance>
         <odometry_frame>odom</odometry_frame>

Commit message: Modify hunter urdf file

File: Workspace/ros2_ws/src/hunter_ros2/hunter_gazebo/urdf/hunter_v1_ntunav_gazebo.xacro (robot description, xacro)
@@ -260,5 +260,5 @@
         <child link="front_right_steer_link"/>
         <axis xyz="0 0 1" rpy="0 0 0" />
-        <dynamics damping="0.0" friction="2"/>
+        <dynamics damping="0.0" friction="1.5"/>
         <limit lower="-0.52" upper="0.52" effort="20" velocity="0.8" />
     </joint>
@@ -270,5 +270,5 @@
         </inertial>
         <visual>
-            <origin xyz="0 ${wheel_steering_offset} 0" rpy="0 0 0" />
+            <origin xyz="0 ${wheel_steering_offset} ${wheel_vertical_offset}" rpy="0 0 0" />
             <geometry>
                 <mesh filename="file://$(find hunter_description)/meshes/steer_conn_fr.dae" />
@@ -277,9 +277,9 @@
     </link>
     <joint name="front_right_wheel" type="continuous">
-        <origin xyz="0 ${wheel_steering_offset} 0" rpy="0 0 0" />
+        <origin xyz="0 ${wheel_steering_offset} ${wheel_vertical_offset}" rpy="0 0 0" />
         <parent link="front_right_steer_link"/>
         <child link="front_right_wheel_link"/>
-        <axis xyz="0 1 0" rpy="0 0 0" />
-        <dynamics damping="0.0" friction="1.0"/>
+        <axis xyz="0 -1 0" rpy="0 0 0" />
+        <dynamics damping="0.0" friction="0"/>
     </joint>
     <link name="front_right_wheel_link">
@@ -308,5 +308,5 @@
         <child link="front_left_steer_link"/>
         <axis xyz="0 0 1" rpy="0 0 0" />
-        <dynamics damping="0.0" friction="2"/>
+        <dynamics damping="0.0" friction="1.5"/>
         <limit lower="-0.52" upper="0.52" effort="20" velocity="0.8" />
     </joint>
@@ -318,5 +318,5 @@
         </inertial>
         <visual>
-            <origin xyz="0 -${wheel_steering_offset} 0" rpy="0 0 0" />
+            <origin xyz="0 -${wheel_steering_offset} ${wheel_vertical_offset}" rpy="0 0 0" />
             <geometry>
                 <mesh filename="file://$(find hunter_description)/meshes/steer_conn_fl.dae" />
@@ -325,9 +325,9 @@
     </link>
     <joint name="front_left_wheel" type="continuous">
-        <origin xyz="0 -${wheel_steering_offset} 0" rpy="0 0 0" />
+        <origin xyz="0 -${wheel_steering_offset} ${wheel_vertical_offset}" rpy="0 0 0" />
         <parent link="front_left_steer_link"/>
         <child link="front_left_wheel_link"/>
-        <axis xyz="0 1 0" rpy="0 0 0" />
-        <dynamics damping="0.0" friction="1.0"/>
+        <axis xyz="0 -1 0" rpy="0 0 0" />
+        <dynamics damping="0.0" friction="0"/>
     </joint>
     <link name="front_left_wheel_link">
@@ -389,5 +389,5 @@
         <parent link="base_link"/>
         <child link="rear_left_wheel_link"/>
-        <dynamics damping="0.0" friction="15"/>
+        <dynamics damping="0.0" friction="5"/>
         <axis xyz="0 1 0" rpy="0 0 0" />
     </joint>
@@ -416,5 +416,5 @@
         <parent link="base_link"/>
         <child link="rear_right_wheel_link"/>
-        <dynamics damping="0.0" friction="15"/>
+        <dynamics damping="0.0" friction="5"/>
         <axis xyz="0 1 0" rpy="0 0 0" />
     </joint>
@@ -435,5 +435,5 @@
         <!-- Max absolute steer angle for tyre in radians-->
         <!-- Any cmd_vel angular z greater than this would be capped -->
-        <max_steer>1.0</max_steer>
+        <max_steer>0.52</max_steer>
         <!-- Max absolute steering angle of steering wheel -->
         <max_steering_angle>0.52</max_steering_angle>
@@ -441,7 +441,7 @@
         <max_speed>1.5</max_speed>
         <!-- PID tuning -->
-        <left_steering_pid_gain>1500 0 1</left_steering_pid_gain>
+        <left_steering_pid_gain>1000 0 1</left_steering_pid_gain>
         <left_steering_i_range>0 0</left_steering_i_range>
-        <right_steering_pid_gain>1500 0 1</right_steering_pid_gain>
+        <right_steering_pid_gain>1000 0 1</right_steering_pid_gain>
         <right_steering_i_range>0 0</right_steering_i_range>
         <linear_velocity_pid_gain>50 0 1</linear_velocity_pid_gain>
